File: hardware/ch55x_bootloader_adapter.kicad_pcb (KiCad board)
At the start: 2 copper layers, 49.4 x 21.2 mm, 7 parts, among them U1 USB-A MALE

Commit message: minor tweaks to adapter, added instructions on back of it
Parts:
- renumbered USB1 to USB-A-F1, U1 to USB-A-M1
Routing:
- net /GND: track 13.0 -> 20.1 mm
Other:
- board text added: "Enter bootloader: Press RESET while holding BOOT key Restart device / exit bootloader: Press RESET"
- board text added: "Insert this adapter to host device (e.g. PC) Insert CH55x device (e.g. Keypad) into receptable"
- board text added: "https://github.com/AmyJeanes/KeypadFlasher"
Changed lines of the file:
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@@
+			)
+		)
+		(property "LCSC" "C149504"
+			(at 0 0 0)
+			(unlocked yes)
+			(layer "F.Fab")
+			(hide yes)
+			(effects
+				(font
+					(size 1 1)
+					(thickness 0.15)
+				)
 			)
 		)
@@
 		(descr "USB-A-TH_U-G-04WD-W-01 footprint")
 		(tags "USB-A-TH_U-G-04WD-W-01 footprint C98125")
-		(property "Reference" "U1"
+		(property "Reference" "USB-A-M1"
 			(at 0 -3 90)
 			(layer "F.SilkS")
@@
 		(descr "USB-A-SMD_U-A-24SS-W-2 footprint")
 		(tags "USB-A-SMD_U-A-24SS-W-2 footprint C530629")
-		(property "Reference" "USB1"
+		(property "Reference" "USB-A-F1"
 			(at 0 -6.237719 90)
 			(layer "F.SilkS")
@@
 	)
 	(gr_text "CH55x Bootloader Adapter"
-		(at 93.4 54 0)
+		(at 93.425 54 0)
 		(layer "F.SilkS")
 		(effects
@@
 			)
 			(justify left bottom)
+		)
+	)
+	(gr_text "Enter bootloader: Press RESET while holding BOOT key\nRestart device / exit bootloader: Press RESET"
+		(at 135.1 68.425 0)
+		(layer "B.SilkS")
+		(effects
+			(font
+				(size 1 1)
+				(thickness 0.2)
+				(bold yes)
+			)
+			(justify left bottom mirror)
+		)
+	)
+	(gr_text "Insert this adapter to host device (e.g. PC)\nInsert CH55x device (e.g. Keypad) into receptable"
+		(at 134.925 57.575 0)
+		(layer "B.SilkS")
+		(effects
+			(font
+				(size 1 1)
+				(thickness 0.2)
+				(bold yes)
+			)
+			(justify left bottom mirror)
+		)
+	)
+	(gr_text "https://github.com/AmyJeanes/KeypadFlasher"
+		(at 122.5 71 0)
+		(layer "B.SilkS")
+		(effects
+			(font
+				(size 1 1)
+				(thickness 0.15)
+			)
+			(justify left bottom mirror)
+		)
+	)
+	(gr_text "CH55x Bootloader Adapter"
+		(at 126 54 0)
+		(layer "B.SilkS")
+		(effects
+			(font
+				(size 1.5 1.5)
+				(thickness 0.1875)
+			)
+			(justify left bottom mirror)
 		)
 	)
@@
 	)
 	(segment
-		(start 127 53.875032)
-		(end 124.424968 53.875032)
-		(width 0.2)
-		(layer "F.Cu")
-		(net 7)
-	)
-	(segment
 		(start 105.34 60.585)
 		(end 103.985 60.585)
@@
 	)
 	(segment
-		(start 126.9746 69.124968)
-		(end 124.424968 69.124968)
+		(start 127 53.875032)
+		(end 133.100076 53.875032)
 		(width 0.2)
 		(layer "F.Cu")
@@
 	)
 	(segment
-		(start 124.424968 69.124968)
-		(end 124.4 69.1)
-		(width 0.2)
-		(layer "F.Cu")
-		(net 7)
-	)
-	(segment
 		(start 103.985 60.585)
 		(end 103.7 60.3)
 		(width 0.2)
 		(layer "F.Cu")
+		(net 7)
+	)
+	(segment
+		(start 126.9746 69.124968)
+		(end 133.074676 69.124968)
+		(width 0.2)
+		(layer "F.Cu")
+		(net 7)
+	)
+	(via
+		(at 130.025 69.124968)
+		(size 0.6)
+		(drill 0.3)
+		(layers "F.Cu" "B.Cu")
 		(net 7)
 	)
@@
 	)
 	(via
-		(at 124.4 69.1)
-		(size 0.6)
-		(drill 0.3)
-		(layers "F.Cu" "B.Cu")
-		(net 7)
-	)
-	(via
 		(at 92.3 67.3)
 		(size 0.6)
@@
 	)
 	(via
-		(at 124.4 53.9)
+		(at 130.05 53.875032)
 		(size 0.6)
 		(drill 0.3)
